File: PulseGenerator.sch (EAGLE design)
At the start: 22 parts, among them IC1 MC34063AD, T1 2N2369, X1 1-227161-0

Commit message: Commit of the current version
Parts:
- removed C2: 220pF, rcl:C-EUC1206
- removed IC1: MC34063AD, v-reg-3:MC34063AD
- removed X1: 1-227161-0, con-coax:1-227161-0
- added GOLD_ORB_SM1: OSHWLOGO_GOLD_ORB_SM, bfl:OSHWLOGO_GOLD_ORB_SM
- added IC2: LT1073-SO08, lt1073:LT1073-SO08
- added LED1: (no value), led:LEDCHIPLED_1206
- added S1: 9450-1, switch-misc:9450-1
- added X2: (no value), con-coax:BU-SMA-H
- C1: device rcl:CPOL-EUC/6032-28R -> rcl:CPOL-EUD/7343-31R
- L1: value DR125 -> 150uH
- R1: value 0.76 -> 220
Connections:
- net GND: now also IC2.GND, IC2.SW2, LED1.C, X2G$1.GND; no longer C2.1, IC1.GND, IC1.SWE, X1.2
- net N$11: now also X2G$1.1; no longer X1.1
- net N$2: now also LED1.A, R1.1; no longer IC1.DRC, R2.2
- net N$3: now also G1.+, S1.P; no longer IC1.IPK, L1.1, R1.2, R2.1
- net N$5: now also IC2.I_LIM, R2.1; no longer C2.2, IC1.TC
- net N$8: now also IC2.SW1; no longer IC1.SWC
- net N$9: now also IC2.FB; no longer IC1.COMP
- net VCC: now also IC2.V_IN, L1.1, R1.2, R2.2, S1.O; no longer G1.+, IC1.VCC, R1.1
Other:
- moved on the sheet: C1, L1, R1, R2, R3, R4
